File: KiCad/Shelly.kicad_pcb (KiCad board)
At the start: 2 copper layers, 14 x 28 mm, 26 parts, among them J1 Shelly 1, J2 Other, J3 USB-C, Q1 PMF170XP,115, Q2 PMF250XNEX, U1 FT231XQ, U2 LMR16006+FB

Commit message: Library update
Routing:
- net Net-(C1-Pad1): track 16.6 -> 15.9 mm
- net +3V3: track 55.8 -> 55.1 mm
- net D-: track 18.7 -> 18.1 mm
Other:
- rule pad_to_mask_clearance: 0 -> 0.01

Commit message: PCB
Parts:
- added ?: , RevK:PasteTasmotizer, F.Cu at (164.1, 95.2)

Commit message: Library update
Parts:
- removed ?: , RevK:PasteTasmotizer
- J3: footprint RevK:USC16-TR-Round -> RevK:USC16-TR
- moved D3 0.14 mm to (171.1, 80.9)
- moved R5 0.14 mm to (171.1, 77.9)
Routing:
- net GND: track 88.2 -> 90.5 mm

Commit message: Minor tweaks
Parts:
- moved R2 0.27 mm to (183.1, 78.2)
- moved R1 0.27 mm to (183.1, 81.1)
Routing:
- net RST: track 28.9 -> 26.6 mm
- net GND: track 90.5 -> 88.8 mm
- net Net-(J3-PadB5): track 6.74 -> 5.90 mm
- net VBUS: track 33.6 -> 33.0 mm
- net Net-(C1-Pad1): track 15.9 -> 15.3 mm
Other:
- board text added: "Invert RTS"

Commit message: Library update
Other:
- board text added: "FTDI: Invert RTS, CBUS0 mode 9"
- board text removed: "Invert RTS"
Changed lines of the file:
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@@
     (effects (font (size 1 1) (thickness 0.15)) (justify right mirror))
   )
-  (gr_text "Invert RTS" (at 183.45 62.45 90) (layer "F.SilkS")
+  (gr_text "GND" (at 183.55 58.6 90) (layer "F.SilkS")
     (effects (font (size 0.5 0.5) (thickness 0.12)))
   )
+  (gr_text "FTDI: Invert RTS, CBUS0 mode 9" (at 183.35 67.3 90) (layer "F.SilkS")
+    (effects (font (size 0.5 0.5) (thickness 0.12)))
+  )

Commit message: Library update
Parts:
- C2: value 0.1uF -> 100nF; footprint RevK:Hidden -> RevK:C_0603_
- C3, C4: footprint RevK:Hidden -> RevK:C_0805_
- D4: footprint RevK:Hidden -> RevK:D_1206_
- L1: footprint RevK:Hidden -> RevK:L_4x4_
- U2: footprint RevK:RegulatorBlockFB -> RevK:SOT-23-Thin-6-Reg

Commit message: Library update
Other:
- rule pad_to_mask_clearance: 0.01 -> 0
Changed lines of the file:
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@@
       (dielectric_constraints no)
     )
-    (pad_to_mask_clearance 0.01)
+    (pad_to_mask_clearance 0)
     (pad_to_paste_clearance_ratio -0.02)
     (pcbplotparams
       (layerselection 0x00010fc_ffffffff)
       (disableapertmacros false)
-      (usegerberextensions false)
+      (usegerberextensions true)
       (usegerberattributes true)
       (usegerberadvancedattributes true)
@@
       (plotinvisibletext false)
       (sketchpadsonfab false)
-      (subtractmaskfromsilk false)
+      (subtractmaskfromsilk true)
       (outputformat 1)
       (mirror false)

Commit message: Production order
Parts:
- D1, D2: footprint Package_TO_SOT_SMD:SOT-363_SC-70-6 -> RevK:SOT-363_SC-70-6-Rot
- J1: footprint Connector_PinHeader_2.54mm:PinHeader_1x05_P2.54mm_Vertical -> RevK:PinHeader_1x05_P2.54mm_Right
- J2: footprint Connector_PinHeader_1.27mm:PinHeader_1x06_P1.27mm_Vertical -> RevK:PinHeader_1x06_P1.27mm_Vertical
- L1: footprint RevK:L_4x4_ -> RevK:L_1210_
- Q1, Q2: footprint Package_TO_SOT_SMD:SOT-323_SC-70 -> RevK:SOT-323_SC-70
- R6: value 100k 1% or 0R -> 100k 1%
- R7: value 30k 1% or NF -> 30k 1%
- U1: footprint RevK:QFN-20-1EP_4x4mm_P0.5mm_EP2.5x2.5mm -> RevK:QFN-20-1EP_4x4mm_P0.5mm_EP2.5x2.5mm-Rot
- U2: value LMR16006+FB -> LMR16006XDDCR; footprint RevK:SOT-23-Thin-6-Reg -> RevK:SOT-23-Thin-6-Reg2
- moved J1 5.20 mm to (177.0, 56.1), turned to 180 degrees
- moved J3 4.40 mm to (177.0, 78.5)
- moved J2 3.17 mm to (179.4, 58.6), turned to 180 degrees
- turned D1 to -90 degrees
- turned D2 to -90 degrees
- turned Q1 to -90 degrees
- turned Q2 to -90 degrees
- turned U1 to 90 degrees
- turned U2 to -90 degrees
