File: PCB/Tas/Tas.kicad_pcb (KiCad board)
At the start: 2 copper layers, 14 x 28 mm, 26 parts, among them J1 Shelly 1, J2 Other, J3 USB-C, Q1 PMF170XP,115, Q2 PMF250XNEX, U1 FT231XQ, U2 LMR16006XDDCR

Commit message: Tidy file structure
Other:
- board text added: "Tasmotizer"
- board text removed: "Shelly Tasmotizer"
Changed lines of the file:
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@@
   (paper "A4")
   (title_block
-    (title "Shelly Tasmotizer")
+    (title "Tasmotizer")
     (date "${DATE}")
     (rev "4")
-    (company "Adrian Kennard Andrews & Arnold Ltd")
-    (comment 1 "www.me.uk")
+    (company "Adrian Kennard, Andrews & Arnold Ltd")
+    (comment 1 "toot.me.uk/@RevK")
+    (comment 2 "www.me.uk")
   )
   (layers
@@
     )
   )
-  (property "DATE" "2023-01-08")
+  (property "DATE" "2023-01-09")
   (net 0 "")
   (net 1 "GND")
@@
     (effects (font (size 1 1) (thickness 0.15)) (justify right mirror))
   )
-  (gr_text "Shelly\nTasmotizer" (at 170.7 60) (layer "B.SilkS")
+  (gr_text "Tasmotizer" (at 170.2 60.8) (layer "B.SilkS")
     (effects (font (size 1 1) (thickness 0.15)) (justify right mirror))
   )

Commit message: Change QR
Parts:
- Art2: footprint RevK:QR-Shelly -> RevK:QR-Tas

Commit message: Put back regulator inductor part
Parts:
- L1: footprint RevK:L_1210_ -> RevK:L_4x4_
- U2: footprint RevK:SOT-23-Thin-6-Reg2 -> RevK:SOT-23-Thin-6-Reg

Commit message: Revised production files
Parts:
- U1: footprint RevK:QFN-20-1EP_4x4mm_P0.5mm_EP2.5x2.5mm-Rot -> RevK:QFN-20-1EP_4x4mm_P0.5mm_EP2.5x2.5mm
- turned U1 to 180 degrees

Commit message: Corrected production files
Parts:
- turned U2 to 0 degrees
Connections:
- U2 pad 1: VBUS -> unconnected-(U2-Pad1)
- U2 pad 2: VBUS -> GND
- U2 pad 3: GND -> Net-(R6-Pad2)
- U2 pad 4: +3V3 -> VBUS
- U2 pad 5: Net-(R6-Pad2) -> VBUS
