File: PCB/Tas/Tas.kicad_pcb (KiCad board)
At the start: 2 copper layers, 28 x 14 mm, 34 parts, among them J1 Shelly 1, J2 Conn_01x07, J3 USB-C-Socket-V, Q1 PMF170XP,115, Q2 PMF250XNEX, U1 FT231XQ, U3 MD8942

Commit message: Comments
Other:
- board text removed: "Fit connector as close to PCB as possible"
Changed lines of the file:
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@@
 		(layer "F.SilkS")
-	)
-	(gr_line
-		(start 76 92)
-		(end 75 91)
-		(stroke
-			(width 0.1)
-			(type default)
-		)
-		(layer "Cmts.User")
-	)
-	(gr_line
-		(start 76 86)
-		(end 76 92)
-		(stroke
-			(width 0.1)
-			(type default)
-		)
-		(layer "Cmts.User")
-	)
-	(gr_line
-		(start 76 92)
-		(end 77 91)
-		(stroke
-			(width 0.1)
-			(type default)
-		)
-		(layer "Cmts.User")
 	)
 	(gr_arc
@@
 			(justify mirror)
 		)
-		(render_cache "2024-03-16" 270
+		(render_cache "2024-03-17" 270
 			(polygon
 				(pts
@@
 			(polygon
 				(pts
-					(xy 104.782597 95.577132) (xy 104.83749 95.588156) (xy 104.88706 95.605897) (xy 104.931143 95.629833)
-					(xy 104.981105 95.670489) (xy 105.020636 95.720006) (xy 105.049351 95.777154) (xy 105.063557 95.824283)
-					(xy 105.071298 95.874492) (xy 105.072787 95.909419) (xy 105.065735 95.96013) (xy 105.054469 96.008826)
-					(xy 105.103143 95.976168) (xy 105.142922 95.947729) (xy 105.183012 95.917496) (xy 105.223014 95.885708)
-					(xy 105.262526 95.852607) (xy 105.301149 95.818433) (xy 105.33848 95.783425) (xy 105.36539 95.756768)
-					(xy 105.411078 95.738466) (xy 105.412773 95.738449) (xy 105.457356 95.760508) (xy 105.468949 95.791694)
-					(xy 105.451679 95.838507) (xy 105.447944 95.842253) (xy 105.403233 95.882602) (xy 105.358155 95.92178)
-					(xy 105.312481 95.959808) (xy 105.265983 95.996706) (xy 105.218432 96.032492) (xy 105.169599 96.067189)
-					(xy 105.119255 96.100815) (xy 105.06717 96.13339) (xy 105.023807 96.158514) (xy 104.976594 96.182985)
-					(xy 104.925507 96.205327) (xy 104.870526 96.224065) (xy 104.811626 96.237722) (xy 104.761671 96.243999)
-					(xy 104.722543 96.245497) (xy 104.662971 96.240141) (xy 104.608075 96.227633) (xy 104.558114 96.208577)
-					(xy 104.513346 96.183575) (xy 104.47403 96.153229) (xy 104.430534 96.105497) (xy 104.397802 96.050764)
-					(xy 104.376446 95.99046) (xy 104.367078 95.926011) (xy 104.366681 95.909419) (xy 104.478789 95.909419)
-					(xy 104.486103 95.965258) (xy 104.507037 96.013982) (xy 104.540074 96.054629) (xy 104.583701 96.086238)
-					(xy 104.636402 96.107847) (xy 104.696662 96.118494) (xy 104.722543 96.119468) (xy 104.779736 96.114078)
-					(xy 104.832971 96.098103) (xy 104.8799 96.071832) (xy 104.918176 96.035557) (xy 104.94545 95.989569)
-					(xy 104.959374 95.934157) (xy 104.96068 95.909419) (xy 104.956258 95.859544) (xy 104.938927 95.805127)
-					(xy 104.909577 95.760101) (xy 104.869382 95.725093) (xy 104.819515 95.700729) (xy 104.761152 95.687635)
-					(xy 104.722543 95.685449) (xy 104.672169 95.689963) (xy 104.614968 95.707386) (xy 104.565685 95.736312)
-					(xy 104.525935 95.775041) (xy 104.497332 95.821874) (xy 104.481493 95.87511) (xy 104.478789 95.909419)
-					(xy 104.366681 95.909419) (xy 104.370295 95.86004) (xy 104.385993 95.796989) (xy 104.413466 95.738616)
-					(xy 104.452001 95.686544) (xy 104.487731 95.652605) (xy 104.528978 95.623811) (xy 104.57544 95.600849)
-					(xy 104.626817 95.584404) (xy 104.682805 95.575162) (xy 104.722543 95.573341)
+					(xy 105.391769 96.231331) (xy 105.347927 96.208063) (xy 105.335837 96.161478) (xy 105.335837 95.713292)
+					(xy 105.282763 95.728948) (xy 105.231538 95.751707) (xy 105.181766 95.779882) (xy 105.133054 95.811783)
+					(xy 105.085006 95.845723) (xy 105.037227 95.880011) (xy 104.989322 95.91296) (xy 104.940896 95.942881)
+					(xy 104.883613 95.972241) (xy 104.824266 95.996461) (xy 104.763174 96.015919) (xy 104.700653 96.030991)
+					(xy 104.637021 96.042057) (xy 104.572597 96.049493) (xy 104.507698 96.053677) (xy 104.442641 96.054988)
+					(xy 104.395267 96.042812) (xy 104.372543 95.999056) (xy 104.395849 95.955081) (xy 104.442641 95.942881)
+					(xy 104.498327 95.941896) (xy 104.554008 95.938667) (xy 104.609402 95.932783) (xy 104.66423 95.92383)
+					(xy 104.718211 95.911396) (xy 104.771063 95.89507) (xy 104.822508 95.874439) (xy 104.872264 95.849091)
+					(xy 104.920188 95.819375) (xy 104.9666 95.787561) (xy 105.011987 95.754746) (xy 105.056834 95.722026)
+					(xy 105.101626 95.690497) (xy 105.146849 95.661256) (xy 105.192988 95.635399) (xy 105.240529 95.614023)
+					(xy 105.289956 95.598224) (xy 105.341756 95.589098) (xy 105.377847 95.587263) (xy 105.424639 95.60526)
+					(xy 105.447573 95.650093) (xy 105.447944 95.657361) (xy 105.447944 96.161478) (xy 105.434603 96.211059)
 				)
 			)
@@
 			)
 		)
-		(render_cache "2024-03-16" 90
+		(render_cache "2024-03-17" 90
 			(polygon
 				(pts
@@
 			(polygon
 				(pts
-					(xy 99.205475 95.017646) (xy 99.255864 95.025964) (xy 99.302103 95.040765) (xy 99.343919 95.061431)
-					(xy 99.381041 95.087345) (xy 99.413198 95.117891) (xy 99.447879 95.164755) (xy 99.472606 95.217291)
-					(xy 99.486733 95.274037) (xy 99.489986 95.318478) (xy 99.489629 95.333411) (xy 99.481198 95.391414)
-					(xy 99.461977 95.445688) (xy 99.432518 95.494948) (xy 99.393372 95.537906) (xy 99.357987 95.565218)
-					(xy 99.317696 95.58772) (xy 99.272731 95.604871) (xy 99.223325 95.616128) (xy 99.16971 95.620948)
-					(xy 99.134495 95.619599) (xy 99.089535 95.613951) (xy 99.036526 95.601659) (xy 98.987042 95.584795)
-					(xy 98.941065 95.564687) (xy 98.898573 95.542663) (xy 98.859546 95.520052) (xy 98.81267 95.490734)
-					(xy 98.76736 95.46047) (xy 98.72341 95.429244) (xy 98.680614 95.397036) (xy 98.638766 95.363828)
-					(xy 98.59766 95.329603) (xy 98.55709 95.294342) (xy 98.516849 95.258028) (xy 98.513488 95.254657)
-					(xy 98.497945 95.212525) (xy 98.508378 95.184458) (xy 98.548503 95.164605) (xy 98.550028 95.16462)
-					(xy 98.591148 95.181091) (xy 98.615367 95.205083) (xy 98.648965 95.23659) (xy 98.683725 95.267347)
-					(xy 98.719286 95.297138) (xy 98.755288 95.325747) (xy 98.79137 95.352957) (xy 98.82717 95.378552)
-					(xy 98.870977 95.407944) (xy 98.860838 95.364118) (xy 98.85449 95.318478) (xy 98.955387 95.318478)
-					(xy 98.956562 95.340742) (xy 98.969094 95.390612) (xy 98.993641 95.432002) (xy 99.028089 95.46465)
-					(xy 99.070325 95.488293) (xy 99.118237 95.502671) (xy 99.16971 95.507522) (xy 99.193003 95.506645)
-					(xy 99.247237 95.497062) (xy 99.294668 95.477615) (xy 99.333932 95.449167) (xy 99.363666 95.412585)
-					(xy 99.382506 95.368733) (xy 99.389089 95.318478) (xy 99.386655 95.2876) (xy 99.3724 95.239687)
-					(xy 99.346658 95.197537) (xy 99.310882 95.162682) (xy 99.266527 95.136648) (xy 99.215047 95.120968)
-					(xy 99.16971 95.116904) (xy 99.134963 95.118872) (xy 99.082435 95.130657) (xy 99.037556 95.152584)
-					(xy 99.00138 95.184092) (xy 98.974965 95.224615) (xy 98.959367 95.27359) (xy 98.955387 95.318478)
-					(xy 98.85449 95.318478) (xy 98.85583 95.287043) (xy 98.862798 95.241855) (xy 98.875583 95.199439)
-					(xy 98.901426 95.148006) (xy 98.937005 95.10344) (xy 98.98197 95.06685) (xy 99.021645 95.045307)
-					(xy 99.066258 95.029341) (xy 99.115662 95.019419) (xy 99.16971 95.016008)
+					(xy 98.567407 95.608199) (xy 98.606865 95.587257) (xy 98.617746 95.545331) (xy 98.617746 95.141964)
+					(xy 98.665513 95.156054) (xy 98.711615 95.176537) (xy 98.756409 95.201894) (xy 98.80025 95.230605)
+					(xy 98.843493 95.261151) (xy 98.886495 95.29201) (xy 98.929609 95.321664) (xy 98.973192 95.348593)
+					(xy 99.024747 95.375018) (xy 99.078159 95.396816) (xy 99.133143 95.414327) (xy 99.189411 95.427893)
+					(xy 99.24668 95.437851) (xy 99.304662 95.444544) (xy 99.363071 95.44831) (xy 99.421622 95.44949)
+					(xy 99.464259 95.438532) (xy 99.48471 95.399151) (xy 99.463735 95.359574) (xy 99.421622 95.348593)
+					(xy 99.371505 95.347707) (xy 99.321392 95.344801) (xy 99.271537 95.339505) (xy 99.222192 95.331447)
+					(xy 99.173609 95.320257) (xy 99.126042 95.305564) (xy 99.079742 95.286996) (xy 99.034961 95.264183)
+					(xy 98.99183 95.237438) (xy 98.950059 95.208806) (xy 98.90921 95.179272) (xy 98.868848 95.149824)
+					(xy 98.828535 95.121448) (xy 98.787835 95.095131) (xy 98.74631 95.07186) (xy 98.703523 95.052621)
+					(xy 98.659039 95.038402) (xy 98.612419 95.030189) (xy 98.579937 95.028537) (xy 98.537824 95.044734)
+					(xy 98.517183 95.085084) (xy 98.516849 95.091625) (xy 98.516849 95.545331) (xy 98.528857 95.589954)
 				)
 			)
@@
 		)
 	)
-	(gr_text "Fit connector as close\nto PCB as possible"
-		(at 69 85 0)
-		(layer "Cmts.User")
-		(effects
-			(font
-				(size 2 2)
-				(thickness 0.15)
-			)
-			(justify left bottom)
-		)
-	)

Commit message: As ordered
Parts:
- added J4: TC2030-USB-NL-DS, RevK:Tag-Connect_TC2030-IDC-NL_2x03_P1.27mm_Vertical, F.Cu at (96.9, 95.5)
- added REF**: Shadow, RevK:Shadow, F.Cu at (100.0, 100.0)
- moved J3 1.39 mm to (103.1, 100.0)
Routing:
- net D+: track 36.8 -> 61.0 mm, vias 2 -> 3
- net GND: track 50.3 -> 40.8 mm, vias 11 -> 13
- net VBUS: track 31.6 -> 34.6 mm, vias 3 -> 4
- net D-: track 29.3 -> 31.7 mm, vias 2 -> 3

Commit message: PCB Update
Parts:
- turned J1 to 180 degrees
Routing:
- net GND: track 40.8 -> 41.9 mm
