File: PCB/Tas/Tas.kicad_sch (KiCad schematic)
At the start: 26 parts, among them J1 Shelly 1, J2 Other, J3 USB-C, Q1 PMF170XP,115, Q2 PMF250XNEX, U1 FT231XQ, U2 LMR16006XDDCR

Commit message: Tidy file structure
Other:
- company: Adrian Kennard Andrews & Arnold Ltd -> Adrian Kennard, Andrews & Arnold Ltd
- title: Shelly Tasmotizer -> Tasmotizer
Changed lines of the file:
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@@
   (paper "A4")
   (title_block
-    (title "Shelly Tasmotizer")
+    (title "Tasmotizer")
     (date "${DATE}")
     (rev "4")
-    (company "Adrian Kennard Andrews & Arnold Ltd")
-    (comment 1 "@TheRealRevK")
+    (company "Adrian Kennard, Andrews & Arnold Ltd")
+    (comment 1 "toot.me.uk/@RevK")
     (comment 2 "www.me.uk")
   )

Commit message: Change QR
Parts:
- Art2: footprint RevK:QR-Shelly -> RevK:QR-Tas
Changed lines of the file:
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@@
       (effects (font (size 1.27 1.27)) hide)
     )
-    (property "Footprint" "RevK:QR-Shelly" (id 2) (at 271.145 173.355 0)
+    (property "Footprint" "RevK:QR-Tas" (id 2) (at 271.145 173.355 0)
       (effects (font (size 1.27 1.27)) hide)
     )
@@
     )
     (path "/00000000-0000-0000-0000-0000610f8780"
-      (reference "Art2") (unit 1) (value "QR") (footprint "RevK:QR-Shelly")
+      (reference "Art2") (unit 1) (value "QR") (footprint "RevK:QR-Tas")
     )
     (path "/00000000-0000-0000-0000-000060815e33"

Commit message: Put back regulator inductor part
Parts:
- L1: footprint RevK:L_1210_ -> RevK:L_4x4_; LCSC Part # C560045 -> C354575
- U2: footprint RevK:SOT-23-Thin-6-Reg2 -> RevK:SOT-23-Thin-6-Reg
Changed lines of the file:
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@@
       (effects (font (size 1.27 1.27)) (justify right))
     )
-    (property "Footprint" "RevK:L_1210_" (id 2) (at 229.235 81.28 0)
+    (property "Footprint" "RevK:L_4x4_" (id 2) (at 229.235 81.28 0)
       (effects (font (size 1.27 1.27)) hide)
     )
@@
       (effects (font (size 1.27 1.27)) hide)
     )
-    (property "LCSC Part #" "C560045" (id 6) (at 229.235 81.28 0)
+    (property "LCSC Part #" "C354575" (id 6) (at 229.235 81.28 0)
       (effects (font (size 1.27 1.27)) hide)
     )
@@
       (effects (font (size 1.27 1.27)) (justify left))
     )
-    (property "Footprint" "RevK:SOT-23-Thin-6-Reg2" (id 2) (at 224.79 73.025 0)
+    (property "Footprint" "RevK:SOT-23-Thin-6-Reg" (id 2) (at 224.79 73.025 0)
       (effects (font (size 1.27 1.27)) hide)
     )
@@
     )
     (path "/0a76536d-55ca-408d-aa7e-dd9e96bca23b"
-      (reference "L1") (unit 1) (value "6.8uH") (footprint "RevK:L_1210_")
+      (reference "L1") (unit 1) (value "6.8uH") (footprint "RevK:L_4x4_")
     )
     (path "/00000000-0000-0000-0000-0000610e7a4f"
@@
     )
     (path "/a372bd78-8214-4035-af04-fcab31e3693f"
-      (reference "U2") (unit 1) (value "LMR16006XDDCR") (footprint "RevK:SOT-23-Thin-6-Reg2")
-    )
-  )
+      (reference "U2") (unit 1) (value "LMR16006XDDCR") (footprint "RevK:SOT-23-Thin-6-Reg")
+    )
+  )

Commit message: Revised production files
Parts:
- U1: footprint RevK:QFN-20-1EP_4x4mm_P0.5mm_EP2.5x2.5mm-Rot -> RevK:QFN-20-1EP_4x4mm_P0.5mm_EP2.5x2.5mm; JLCPCB Rotation Offset (none) -> 90
Changed lines of the file:
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@@
     (property "Reference" "U1" (id 0) (at 130.81 142.24 0))
     (property "Value" "FT231XQ" (id 1) (at 143.51 120.65 0))
-    (property "Footprint" "RevK:QFN-20-1EP_4x4mm_P0.5mm_EP2.5x2.5mm-Rot" (id 2) (at 177.8 140.97 0)
+    (property "Footprint" "RevK:QFN-20-1EP_4x4mm_P0.5mm_EP2.5x2.5mm" (id 2) (at 177.8 140.97 0)
       (effects (font (size 1.27 1.27)) hide)
     )
@@
     )
     (property "LCSC Part #" "C132159" (id 6) (at 143.51 120.65 0)
+      (effects (font (size 1.27 1.27)) hide)
+    )
+    (property "JLCPCB Rotation Offset" "90" (id 7) (at 143.51 120.65 0)
       (effects (font (size 1.27 1.27)) hide)
     )
@@
     )
     (path "/00000000-0000-0000-0000-0000607d3e37"
-      (reference "U1") (unit 1) (value "FT231XQ") (footprint "RevK:QFN-20-1EP_4x4mm_P0.5mm_EP2.5x2.5mm-Rot")
+      (reference "U1") (unit 1) (value "FT231XQ") (footprint "RevK:QFN-20-1EP_4x4mm_P0.5mm_EP2.5x2.5mm")
     )
     (path "/a372bd78-8214-4035-af04-fcab31e3693f"

Commit message: Corrected production files
Parts:
- removed U2: LMR16006XDDCR, RevK:SOT-23-Thin-6-Reg, symbol RevK:LMR16006+FB
- added U2: LMR16006XDDCR, RevK:SOT-23-Thin-6-Reg, symbol RevK:LMR16006XDDCR
- U1: JLCPCB Rotation Offset 90 -> -90
Connections:
- net +3V3: now also U2.7 (VOUT)
- net GND: now also U2.2 (GND)
- net VBUS: now also U2.4 (SHDN), U2.5 (VIN)
- net at R6.2, R7.2: now also U2.3 (FB)

Commit message: Revised PCB with 7 pin small connector
Parts:
- removed J2: Other, RevK:PinHeader_1x06_P1.27mm_Vertical, symbol Connector_Generic:Conn_01x06
- added J2: Conn_01x07, RevK:PinHeader_1x07_P1.27mm_Vertical, symbol Connector_Generic:Conn_01x07
Connections:
- net +3V3: now also J2.4 (Pin_4)
- net GND: now also J2.1 (Pin_1)
- net GPIO0: now also J2.2 (Pin_2)
- net RXD: now also J2.5 (Pin_5)
- net TXD: now also J2.6 (Pin_6)
- net at J1.3 (Pin_3), Q1.3 (D), Q2.3 (D): now also J2.3 (Pin_3)
- no-connect marks 3 -> 4
Changed lines of the file:
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@@
   (junction (at 138.43 83.82) (diameter 0) (color 0 0 0 0)
   )
+  (no_connect (at 68.58 80.01))
   (no_connect (at 161.29 130.81))
   (no_connect (at 161.29 133.35))
@@
     (pin "5")
   )
-  (symbol (lib_id "Connector_Generic:Conn_01x06") (at 73.66 69.85 0) (unit 1)
-    (in_bom yes) (on_board yes)
-    (property "Reference" "J2" (id 0) (at 72.39 60.96 0)
-      (effects (font (size 1.27 1.27)) (justify left))
-    )
-    (property "Value" "Other" (id 1) (at 75.692 72.3646 0)
-      (effects (font (size 1.27 1.27)) (justify left))
-    )
-    (property "Footprint" "RevK:PinHeader_1x06_P1.27mm_Vertical" (id 2) (at 73.66 69.85 0)
-      (effects (font (size 1.27 1.27)) hide)
-    )
-    (property "Datasheet" "~" (id 3) (at 73.66 69.85 0)
-      (effects (font (size 1.27 1.27)) hide)
-    )
-    (property "LCSC Part #" "C2832273" (id 4) (at 73.66 69.85 0)
-      (effects (font (size 1.27 1.27)) hide)
-    )
-    (pin "1")
-    (pin "2")
-    (pin "3")
-    (pin "4")
-    (pin "5")
-    (pin "6")
-  )
   (symbol (lib_id "power:GND") (at 68.58 64.77 270) (unit 1)
     (in_bom yes) (on_board yes)
@@
     (pin "~")
   )
+  (symbol (lib_id "Connector_Generic:Conn_01x07") (at 73.66 72.39 0) (unit 1)
+    (in_bom yes) (on_board yes) (fields_autoplaced)
+    (property "Reference" "J2" (id 0) (at 75.692 71.5553 0)
+      (effects (font (size 1.27 1.27)) (justify left))
+    )
+    (property "Value" "Conn_01x07" (id 1) (at 75.692 74.0922 0)
+      (effects (font (size 1.27 1.27)) (justify left))
+    )
+    (property "Footprint" "RevK:PinHeader_1x07_P1.27mm_Vertical" (id 2) (at 73.66 72.39 0)
+      (effects (font (size 1.27 1.27)) hide)
+    )
+    (property "Datasheet" "~" (id 3) (at 73.66 72.39 0)
+      (effects (font (size 1.27 1.27)) hide)
+    )
+    (property "LCSC Part #" "C2832274" (id 4) (at 73.66 72.39 0)
+      (effects (font (size 1.27 1.27)) hide)
+    )
+    (pin "1")
+    (pin "2")
+    (pin "3")
+    (pin "4")
+    (pin "5")
+    (pin "6")
+    (pin "7")
+  )
   (symbol (lib_id "RevK:Hidden") (at 229.235 77.47 0) (unit 1)
     (in_bom yes) (on_board yes)
@@
       (reference "J1") (unit 1) (value "Shelly 1") (footprint "RevK:PinHeader_1x05_P2.54mm_Right")
     )
-    (path "/00000000-0000-0000-0000-0000607b65bb"
-      (reference "J2") (unit 1) (value "Other") (footprint "RevK:PinHeader_1x06_P1.27mm_Vertical")
+    (path "/2f7812a2-f996-4689-9055-d1875d2cc709"
+      (reference "J2") (unit 1) (value "Conn_01x07") (footprint "RevK:PinHeader_1x07_P1.27mm_Vertical")
     )
     (path "/00000000-0000-0000-0000-000060436927"

Commit message: Library update
Parts:
- U2: value LMR16006XDDCR -> LMR16006YDDCR; JLCPCB Rotation Offset 90 -> 0; LCSC Part # C87080 -> C290195; Part No LMR16006XDDCR -> LMR16006YDDCR
Changed lines of the file:
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@@
     (in_bom yes) (on_board yes) (fields_autoplaced)
     (property "Reference" "U2" (id 0) (at 231.14 70.7222 0))
-    (property "Value" "LMR16006XDDCR" (id 1) (at 231.14 73.2591 0))
+    (property "Value" "LMR16006YDDCR" (id 1) (at 231.14 73.2591 0))
     (property "Footprint" "RevK:SOT-23-Thin-6-Reg" (id 2) (at 228.6 92.075 0)
       (effects (font (size 1.27 1.27)) hide)
@@
       (effects (font (size 1.27 1.27)) hide)
     )
-    (property "Part No" "LMR16006XDDCR" (id 5) (at 231.775 90.17 0)
+    (property "Part No" "LMR16006YDDCR" (id 5) (at 231.775 90.17 0)
       (effects (font (size 1.27 1.27)) hide)
     )
-    (property "LCSC Part #" "C87080" (id 6) (at 219.075 90.17 0)
+    (property "LCSC Part #" "C290195" (id 6) (at 219.075 90.17 0)
       (effects (font (size 1.27 1.27)) hide)
     )
-    (property "JLCPCB Rotation Offset" "90" (id 7) (at 243.84 90.17 0)
+    (property "JLCPCB Rotation Offset" "0" (id 7) (at 243.84 90.17 0)
       (effects (font (size 1.27 1.27)) hide)
     )
@@
     )
     (path "/ff65da73-9ec3-453c-8cfa-18c86da48974"
-      (reference "U2") (unit 1) (value "LMR16006XDDCR") (footprint "RevK:SOT-23-Thin-6-Reg")
+      (reference "U2") (unit 1) (value "LMR16006YDDCR") (footprint "RevK:SOT-23-Thin-6-Reg")
     )
   )

Commit message: Tweak
Parts:
- J2: JLCPCB Rotation Offset (none) -> 90
- J3: JLCPCB Rotation Offset (none) -> 0
- U2: JLCPCB Rotation Offset 0 -> 180
Changed lines of the file:
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@@
+      (effects (font (size 1.27 1.27)) hide)
+    )
+    (property "JLCPCB Rotation Offset" "0" (id 7) (at 138.43 60.96 0)
       (effects (font (size 1.27 1.27)) hide)
     )
@@
       (effects (font (size 1.27 1.27)) hide)
     )
+    (property "JLCPCB Rotation Offset" "90" (id 5) (at 73.66 72.39 0)
+      (effects (font (size 1.27 1.27)) hide)
+    )
     (pin "1")
     (pin "2")
@@
       (effects (font (size 1.27 1.27)) hide)
     )
-    (property "JLCPCB Rotation Offset" "0" (id 7) (at 243.84 90.17 0)
-      (effects (font (size 1.27 1.27)) hide)
-    )
+    (property "JLCPCB Rotation Offset" "180" (id 7) (at 243.84 90.17 0)
+      (effects (font (size 1.27 1.27)) hide)
+    )
