File: PCB/ShellyPower/ShellyPower.kicad_pcb (KiCad board)
At the start: 2 copper layers, 110 x 45 mm, 20 parts, among them J1 Shelly 1, J2 Conn_01x07, J3 USB-C, U2 LMR16006XDDCR

Commit message: Production files
Changed lines of the file:
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@@
     (descr "surface-mounted straight pin header, 1x05, 2.54mm pitch, single row, style 2 (pin 1 right)")
     (tags "Surface mounted pin header SMD 1x05 2.54mm single row style2 pin1 right")
-    (property "LCSC Part #" "C225491")
+    (property "JLCPCB Rotation Offset" "-90")
+    (property "LCSC Part #" "C780063")
     (property "Sheetfile" "ShellyPower.kicad_sch")
     (property "Sheetname" "")
     (attr smd)
-    (fp_text reference "J1" (at 0 -7.41 90) (layer "F.SilkS")
+    (fp_text reference "J1" (at 0 -7.41 90) (layer "F.SilkS") hide
       (effects (font (size 1 1) (thickness 0.15)))
     )

Commit message: Tweak to fit SHelly 1 better
Other:
- board text added: "3.3V power supply"
- board text removed: "Shelly power supply"
Changed lines of the file:
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@@
     (effects (font (size 1 1) (thickness 0.15)) (justify mirror))
   )
-  (gr_text "Shelly power supply" (at 210.1 87.8) (layer "F.SilkS")
+  (gr_text "3.3V power supply" (at 210.1 87.8) (layer "F.SilkS")
     (effects (font (size 2 2) (thickness 0.3)))
   )
