File: PCB/ShellyPower/ShellyPower.kicad_pcb (KiCad board)
At the start: 2 copper layers, 110 x 45 mm, 20 parts, among them J1 Shelly 1, J2 Conn_01x07, J3 USB-C, U2 LMR16006XDDCR

Commit message: PCB Update
Parts:
- removed Art2: QR, RevK:QR-Tas
- J3: footprint RevK:USC16-TR -> RevK:USB-C-Socket-H
- moved J3 1.65 mm to (161.0, 73.2)
Connections:
- J3 pad A6: unconnected-(J3-PadA6) -> unconnected-(J3-D+-PadA6)_1
- J3 pad A7: unconnected-(J3-PadA7) -> unconnected-(J3-D--PadA7)_1
- J3 pad B6: unconnected-(J3-PadA6) -> unconnected-(J3-D+-PadA6)
- J3 pad B7: unconnected-(J3-PadA7) -> unconnected-(J3-D--PadA7)
Routing:
- net GND: track 7.34 -> 21.7 mm
