File: PCB/ShellyPower/ShellyPower.kicad_sch (KiCad schematic)
At the start: 20 parts, among them J1 Shelly 1, J2 Conn_01x07, J3 USB-C, U2 LMR16006XDDCR

Commit message: Production files
Parts:
- J1: JLCPCB Rotation Offset (none) -> -90; LCSC Part # C225491 -> C780063
Changed lines of the file:
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@@
       (effects (font (size 1.27 1.27)) hide)
     )
-    (property "LCSC Part #" "C225491" (id 4) (at 139.7 110.49 0)
+    (property "LCSC Part #" "C780063" (id 4) (at 139.7 110.49 0)
       (effects (font (size 1.27 1.27)) hide)
     )
+    (property "JLCPCB Rotation Offset" "-90" (id 5) (at 139.7 110.49 0)
+      (effects (font (size 1.27 1.27)) hide)
+    )

Commit message: PCB Update
Parts:
- removed Art2: QR, RevK:QR-Tas, symbol RevK:QR
- C2: LCSC Part # C30926 -> (none); MPN (none) -> C30926
- C3: LCSC Part # C19110 -> (none); MPN (none) -> C19110
- C4: LCSC Part # C17024 -> (none); MPN (none) -> C17024
- D4: LCSC Part # C143805 -> (none); MPN (none) -> C143805
- J1: JLCPCB Rotation Offset -90 -> (none); LCSC Part # C780063 -> (none); MPN (none) -> C780063
- J2: LCSC Part # C2832274 -> (none); MPN (none) -> C2832274
- J3: value USB-C -> USB-C-Socket-V; footprint RevK:USC16-TR -> RevK:USB-C-Socket-H; symbol RevK:USB-C -> RevK:USB-C-Socket-H; LCSC Part # C709357 -> (none); MPN (none) -> C709357
- L1: LCSC Part # C354575 -> (none); MPN (none) -> C354575
- R6: LCSC Part # C14675 -> (none); MPN (none) -> C14675
- R7: LCSC Part # C100001 -> (none); MPN (none) -> C100001
- U2: JLCPCB Rotation Offset 90 -> (none); LCSC Part # C87080 -> (none); MPN (none) -> C87080
