File: PCB/Tas2/Tas2.kicad_pcb (KiCad board)
At the start: 2 copper layers, 14 x 28 mm, 27 parts, among them J1 Shelly 1, J2 Conn_01x07, J3 USB-C, Q1 PMF170XP,115, Q3 BSD235C, U2 LMR16006YDDCR, U3 CH340X

Commit message: Ooops, try again for order
Parts:
- removed Q3: BSD235C, RevK:SOT-363_SC-70-6
- added Q2: 2N7002BKS, RevK:SOT-363_SC-70-6, F.Cu at (174.9, 61.2)
Connections:
- U3 pad 1: D- -> D+
- U3 pad 2: D+ -> D-
Routing:
- net GND: track 93.9 -> 98.9 mm
- net RXD: track 51.9 -> 48.0 mm
- net Net-(Q1-G): track 6.80 -> 4.89 mm
- net D-: track 17.0 -> 18.9 mm
- net Net-(J1-Pin_3): track 15.9 -> 14.3 mm
- net D+: track 18.7 -> 20.1 mm
- net GPIO0: track 18.2 -> 19.4 mm
- net RST: track 16.0 -> 15.5 mm

Commit message: GND CTS
Connections:
- U3 pad 5: unconnected-(U3-~{CTS}-Pad5) -> GND
Routing:
- net GND: track 98.9 -> 101.1 mm
