File: PCB/Tas2/Tas2.kicad_pcb (KiCad board)
At the start: 2 copper layers, 14 x 28 mm, 27 parts, among them J1 Shelly 1, J2 Conn_01x07, J3 USB-C, Q1 PMF170XP,115, Q2 2N7002BKS, U2 LMR16006YDDCR, U3 CH340X

Commit message: Corrected USB circuit, grrr
Parts:
- removed R3, R4: 27R, RevK:R_0603
- moved C5 9.98 mm to (182.7, 64.8), turned to -90 degrees
Connections:
- J3 pad A6: Net-(J3-D+-PadA6) -> D+
- J3 pad A7: Net-(J3-D--PadA7) -> D-
- J3 pad B6: Net-(J3-D+-PadA6) -> D+
- J3 pad B7: Net-(J3-D--PadA7) -> D-
- U3 pad 10: VBUS -> +3V3
- U3 pad 7: VBUS -> +3V3
Routing:
- net VBUS: track 39.1 -> 14.5 mm, vias 2 -> 0
- net +3V3: track 55.6 -> 71.3 mm
- net D-: track 18.9 -> 28.5 mm
- net Net-(J3-D--PadA7): track 9.05 -> 0.00 mm
- net D+: track 20.1 -> 28.5 mm, vias 2 -> 3
- net Net-(J3-D+-PadA6): track 7.89 -> 0.00 mm, vias 2 -> 0
- net GND: track 101.1 -> 100.7 mm, vias 7 -> 8
Other:
- board text added: "A"
