File: PCB/Tas2/Tas2.kicad_sch (KiCad schematic)
At the start: 27 parts, among them J1 Shelly 1, J2 Conn_01x07, J3 USB-C, Q1 PMF170XP,115, Q3 BSD235C, U2 LMR16006YDDCR, U3 CH340X

Commit message: For order
Parts:
- Q3: JLCPCB Rotation Offset (none) -> 180
Changed lines of the file:
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@@
+      (effects (font (size 1.27 1.27)) hide)
+    )
+    (property "JLCPCB Rotation Offset" "180" (at 38.735 68.58 0)
       (effects (font (size 1.27 1.27)) hide)
     )
@@
       (effects (font (size 1.27 1.27)) hide)
     )
+    (property "JLCPCB Rotation Offset" "180" (at 59.055 73.66 0)
+      (effects (font (size 1.27 1.27)) hide)
+    )

Commit message: Ooops, try again for order
Parts:
- removed Q3: BSD235C, RevK:SOT-363_SC-70-6, symbol Transistor_FET:BSD235C
- added Q2: 2N7002BKS, RevK:SOT-363_SC-70-6, symbol Transistor_FET:FDG1024NZ
Connections:
- net D+: now also U3.1 (UD+); no longer U3.2 (UD-)
- net D-: now also U3.2 (UD-); no longer U3.1 (UD+)
- net GND: now also Q2.1 (S), Q2.4 (S)
- net RST: now also Q2.2 (G)
- net at J1.3 (Pin_3), J2.3 (Pin_3), Q1.3 (D): now also Q2.3 (D)
- net at Q1.1 (G), R9.2: now also Q2.5 (G), Q2.6 (D)

Commit message: GND CTS
Connections:
- net GND: now also U3.5 (~{CTS})
- no-connect marks 2 -> 1
Changed lines of the file:
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@@
   )
   (no_connect (at 88.9 73.66))
-  (no_connect (at 144.145 139.7))
   (wire (pts (xy 130.81 83.82) (xy 138.43 83.82))
     (stroke (width 0) (type default))
@@
         )
       )
+    )
+  )
+  (symbol (lib_id "power:GND") (at 144.145 139.7 90) (unit 1)
+    (in_bom yes) (on_board yes) (dnp no)
+    (property "Reference" "#PWR016" (at 150.495 139.7 0)
+      (effects (font (size 1.27 1.27)) hide)
+    )
+    (property "Value" "GND" (at 148.5392 139.573 0)
+      (effects (font (size 1.27 1.27)))
+    )
+    (property "Footprint" "" (at 144.145 139.7 0)
+      (effects (font (size 1.27 1.27)) hide)
+    )
+    (property "Datasheet" "" (at 144.145 139.7 0)
+      (effects (font (size 1.27 1.27)) hide)
+    )
+    (pin "1")
+    (instances
+      (project "Tas2"
+        (path "/42713045-fffd-4b2d-ae1e-7232d705fb12"
+          (reference "#PWR016") (unit 1)
+        )
+      )

Commit message: Corrected USB circuit, grrr
Parts:
- removed R3, R4: 27R, RevK:R_0603, symbol Device:R
Connections:
- net +3V3: now also U3.10 (V3), U3.7 (VCC)
- net D+: now also J3.A6 (D+), J3.B6 (D+)
- net D-: now also J3.A7 (D-), J3.B7 (D-)
- net VBUS: no longer U3.10 (V3), U3.7 (VCC)
Other:
- moved on the sheet: C5
Changed lines of the file:
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@@
-    (stroke (width 0) (type default))
-  )
-  (wire (pts (xy 179.07 60.96) (xy 184.15 60.96))
     (stroke (width 0) (type default))
   )
@@
     (stroke (width 0) (type default))
   )
-  (wire (pts (xy 153.67 63.5) (xy 171.45 63.5))
-    (stroke (width 0) (type default))
-  )
   (wire (pts (xy 213.36 85.725) (xy 213.36 88.9))
     (stroke (width 0) (type default))
@@
     (stroke (width 0) (type default))
   )
-  (wire (pts (xy 179.07 63.5) (xy 184.15 63.5))
-    (stroke (width 0) (type default))
-  )
   (wire (pts (xy 168.91 52.07) (xy 163.83 52.07))
     (stroke (width 0) (type default))
   )
   (wire (pts (xy 144.145 127) (xy 147.955 127))
-    (stroke (width 0) (type default))
-  )
-  (wire (pts (xy 153.67 60.96) (xy 171.45 60.96))
     (stroke (width 0) (type default))
   )
@@
     )
   )
-  (global_label "D-" (shape input) (at 123.825 138.43 180) (fields_autoplaced)
+  (global_label "D-" (shape bidirectional) (at 123.825 138.43 180) (fields_autoplaced)
     (effects (font (size 1.27 1.27)) (justify right))
-    (property "Intersheetrefs" "${INTERSHEET_REFS}" (at -28.575 38.1 0)
-      (effects (font (size 1.27 1.27)) hide)
+    (property "Intersheetrefs" "${INTERSHEET_REFS}" (at 117.7785 138.43 0)
+      (effects (font (size 1.27 1.27)) (justify right) hide)
     )
   )
@@
     )
   )
-  (global_label "D-" (shape input) (at 184.15 60.96 0) (fields_autoplaced)
+  (global_label "D-" (shape bidirectional) (at 153.67 60.96 0) (fields_autoplaced)
     (effects (font (size 1.27 1.27)) (justify left))
-    (property "Intersheetrefs" "${INTERSHEET_REFS}" (at -25.4 15.24 0)
-      (effects (font (size 1.27 1.27)) hide)
+    (property "Intersheetrefs" "${INTERSHEET_REFS}" (at 159.7165 60.96 0)
+      (effects (font (size 1.27 1.27)) (justify left) hide)
     )
   )
@@
     )
   )
-  (global_label "D+" (shape input) (at 123.825 135.89 180) (fields_autoplaced)
+  (global_label "D+" (shape bidirectional) (at 123.825 135.89 180) (fields_autoplaced)
     (effects (font (size 1.27 1.27)) (justify right))
-    (property "Intersheetrefs" "${INTERSHEET_REFS}" (at -28.575 33.02 0)
-      (effects (font (size 1.27 1.27)) hide)
+    (property "Intersheetrefs" "${INTERSHEET_REFS}" (at 117.7785 135.89 0)
+      (effects (font (size 1.27 1.27)) (justify right) hide)
     )
   )
@@
     )
   )
-  (global_label "VBUS" (shape input) (at 133.985 120.015 90) (fields_autoplaced)
-    (effects (font (size 1.27 1.27)) (justify left))
-    (property "Intersheetrefs" "${INTERSHEET_REFS}" (at -33.655 34.925 0)
-      (effects (font (size 1.27 1.27)) hide)
-    )
-  )
   (global_label "RXD" (shape input) (at 79.375 168.275 270) (fields_autoplaced)
     (effects (font (size 1.27 1.27)) (justify right))
@@
     )
   )
-  (global_label "D+" (shape input) (at 184.15 63.5 0) (fields_autoplaced)
+  (global_label "D+" (shape bidirectional) (at 153.67 63.5 0) (fields_autoplaced)
     (effects (font (size 1.27 1.27)) (justify left))
-    (property "Intersheetrefs" "${INTERSHEET_REFS}" (at -25.4 12.7 0)
-      (effects (font (size 1.27 1.27)) hide)
+    (property "Intersheetrefs" "${INTERSHEET_REFS}" (at 159.7165 63.5 0)
+      (effects (font (size 1.27 1.27)) (justify left) hide)
     )
   )
@@
     )
   )
-  (symbol (lib_id "Device:R") (at 175.26 60.96 90) (unit 1)
-    (in_bom yes) (on_board yes) (dnp no)
-    (property "Reference" "R3" (at 175.26 58.42 90)
-      (effects (font (size 1.27 1.27)))
-    )
-    (property "Value" "27R" (at 175.26 60.96 90)
-      (effects (font (size 1.27 1.27)))
-    )
-    (property "Footprint" "RevK:R_0603" (at 175.26 62.738 90)
-      (effects (font (size 1.27 1.27)) hide)
-    )
-    (property "Datasheet" "~" (at 175.26 60.96 0)
-      (effects (font (size 1.27 1.27)) hide)
-    )
-    (pin "1")
-    (pin "2")
-    (instances
-      (project "Tas2"
-        (path "/42713045-fffd-4b2d-ae1e-7232d705fb12"
-          (reference "R3") (unit 1)
-        )
-      )
-    )
-  )
-  (symbol (lib_id "Device:R") (at 175.26 63.5 90) (unit 1)
-    (in_bom yes) (on_board yes) (dnp no)
-    (property "Reference" "R4" (at 175.26 66.04 90)
-      (effects (font (size 1.27 1.27)))
-    )
-    (property "Value" "27R" (at 175.26 63.5 90)
-      (effects (font (size 1.27 1.27)))
-    )
-    (property "Footprint" "RevK:R_0603" (at 175.26 65.278 90)
-      (effects (font (size 1.27 1.27)) hide)
-    )
-    (property "Datasheet" "~" (at 175.26 63.5 0)
-      (effects (font (size 1.27 1.27)) hide)
-    )
-    (pin "1")
-    (pin "2")
-    (instances
-      (project "Tas2"
-        (path "/42713045-fffd-4b2d-ae1e-7232d705fb12"
-          (reference "R4") (unit 1)
-        )
-      )
-    )
-  )
   (symbol (lib_id "Connector_Generic:Conn_01x05") (at 93.98 36.83 0) (unit 1)
     (in_bom yes) (on_board yes) (dnp no)
@@
     )
   )
-  (symbol (lib_id "power:GND") (at 201.295 130.81 0) (unit 1)
+  (symbol (lib_id "power:GND") (at 118.745 122.555 0) (unit 1)
     (in_bom yes) (on_board yes) (dnp no) (fields_autoplaced)
-    (property "Reference" "#PWR026" (at 201.295 137.16 0)
-      (effects (font (size 1.27 1.27)) hide)
-    )
-    (property "Value" "GND" (at 201.295 135.2534 0)
-      (effects (font (size 1.27 1.27)))
-    )
-    (property "Footprint" "" (at 201.295 130.81 0)
-      (effects (font (size 1.27 1.27)) hide)
-    )
-    (property "Datasheet" "" (at 201.295 130.81 0)
+    (property "Reference" "#PWR026" (at 118.745 128.905 0)
+      (effects (font (size 1.27 1.27)) hide)
+    )
+    (property "Value" "GND" (at 118.745 126.9984 0)
+      (effects (font (size 1.27 1.27)))
+    )
+    (property "Footprint" "" (at 118.745 122.555 0)
+      (effects (font (size 1.27 1.27)) hide)
+    )
+    (property "Datasheet" "" (at 118.745 122.555 0)
       (effects (font (size 1.27 1.27)) hide)
     )
@@
         (path "/42713045-fffd-4b2d-ae1e-7232d705fb12"
           (reference "#PWR016") (unit 1)
+        )
+      )
+    )
+  )
+  (symbol (lib_id "power:+3.3V") (at 133.985 120.015 0) (unit 1)
+    (in_bom yes) (on_board yes) (dnp no)
+    (property "Reference" "#PWR017" (at 133.985 123.825 0)
+      (effects (font (size 1.27 1.27)) hide)
+    )
+    (property "Value" "+3.3V" (at 134.366 116.7638 90)
+      (effects (font (size 1.27 1.27)) (justify left))
+    )
+    (property "Footprint" "" (at 133.985 120.015 0)
+      (effects (font (size 1.27 1.27)) hide)
+    )
+    (property "Datasheet" "" (at 133.985 120.015 0)
+      (effects (font (size 1.27 1.27)) hide)
+    )
+    (pin "1")
+    (instances
+      (project "Tas2"
+        (path "/42713045-fffd-4b2d-ae1e-7232d705fb12"
+          (reference "#PWR017") (unit 1)
         )
       )
@@
     )
   )
-  (symbol (lib_id "power:+3.3V") (at 201.295 123.19 0) (unit 1)
+  (symbol (lib_id "power:+3.3V") (at 118.745 114.935 0) (unit 1)
     (in_bom yes) (on_board yes) (dnp no) (fields_autoplaced)
-    (property "Reference" "#PWR025" (at 201.295 127 0)
-      (effects (font (size 1.27 1.27)) hide)
-    )
-    (property "Value" "+3.3V" (at 201.295 119.6142 0)
-      (effects (font (size 1.27 1.27)))
-    )
-    (property "Footprint" "" (at 201.295 123.19 0)
-      (effects (font (size 1.27 1.27)) hide)
-    )
-    (property "Datasheet" "" (at 201.295 123.19 0)
+    (property "Reference" "#PWR025" (at 118.745 118.745 0)
+      (effects (font (size 1.27 1.27)) hide)
+    )
+    (property "Value" "+3.3V" (at 118.745 111.3592 0)
+      (effects (font (size 1.27 1.27)))
+    )
+    (property "Footprint" "" (at 118.745 114.935 0)
+      (effects (font (size 1.27 1.27)) hide)
+    )
+    (property "Datasheet" "" (at 118.745 114.935 0)
       (effects (font (size 1.27 1.27)) hide)
     )
@@
     )
   )
-  (symbol (lib_id "Device:C") (at 201.295 127 0) (unit 1)
+  (symbol (lib_id "Device:C") (at 118.745 118.745 0) (unit 1)
     (in_bom yes) (on_board yes) (dnp no) (fields_autoplaced)
-    (property "Reference" "C5" (at 204.216 126.1653 0)
-      (effects (font (size 1.27 1.27)) (justify left))
-    )
-    (property "Value" "100nF" (at 204.216 128.7022 0)
-      (effects (font (size 1.27 1.27)) (justify left))
-    )
-    (property "Footprint" "RevK:C_0603" (at 202.2602 130.81 0)
-      (effects (font (size 1.27 1.27)) hide)
-    )
-    (property "Datasheet" "~" (at 201.295 127 0)
-      (effects (font (size 1.27 1.27)) hide)
-    )
+    (property "Reference" "C5" (at 121.666 117.9103 0)
+      (effects (font (size 1.27 1.27)) (justify left))
+    )
+    (property "Value" "100nF" (at 121.666 120.4472 0)
+      (effects (font (size 1.27 1.27)) (justify left))
+    )
+    (property "Footprint" "RevK:C_0603" (at 119.7102 122.555 0)
+      (effects (font (size 1.27 1.27)) hide)
+    )
+    (property "Datasheet" "~" (at 118.745 118.745 0)
+      (effects (font (size 1.27 1.27)) hide)
+    )
