File: PCB/Tas3/Tas.kicad_sch (KiCad schematic)
At the start: 28 parts, among them J1 Shelly 1, J2 Conn_01x07, J3 USB-C, Q1 AP2003, U1 MD8942, U2 74LVC1G07, U3 CH340X, U4 74LVC1G06SE-7

Commit message: FFS
Parts:
- added C3: 100nF, RevK:C_0402, symbol Device:C
- added C4: 22uF, RevK:C_0402, symbol Device:C
- C2: value 100nF -> 10nF
Connections:
- net GND: now also C3.1, C4.1
- net VBUS: now also C3.2, C4.2
Other:
- note added: "Still not fucking working"
- moved on the sheet: C2
Changed lines of the file:
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@@
   (junction (at 134.62 70.485) (diameter 0) (color 0 0 0 0)
   )
+  (junction (at 151.765 106.045) (diameter 0) (color 0 0 0 0)
+  )
   (junction (at 150.495 131.445) (diameter 0) (color 0 0 0 0)
+  )
+  (junction (at 146.05 106.045) (diameter 0) (color 0 0 0 0)
   )
   (junction (at 239.395 113.03) (diameter 0) (color 0 0 0 0)
@@
     (stroke (width 0) (type default))
   )
-  (wire (pts (xy 139.065 103.505) (xy 139.065 109.855))
+  (wire (pts (xy 132.08 109.855) (xy 139.065 109.855))
+    (stroke (width 0) (type default))
+  )
+  (wire (pts (xy 146.05 109.855) (xy 141.605 109.855))
+    (stroke (width 0) (type default))
+  )
+  (wire (pts (xy 132.08 103.505) (xy 132.08 109.855))
     (stroke (width 0) (type default))
   )
@@
     (stroke (width 0) (type default))
   )
+  (wire (pts (xy 146.05 103.505) (xy 146.05 106.045))
+    (stroke (width 0) (type default))
+  )
   (wire (pts (xy 247.015 118.11) (xy 247.015 123.19))
     (stroke (width 0) (type default))
   )
+  (wire (pts (xy 146.05 106.045) (xy 151.765 106.045))
+    (stroke (width 0) (type default))
+  )
+  (wire (pts (xy 151.765 106.045) (xy 156.845 106.045))
+    (stroke (width 0) (type default))
+  )
   (wire (pts (xy 153.67 40.005) (xy 156.21 40.005))
     (stroke (width 0) (type default))
@@
     (stroke (width 0) (type default))
   )
+  (wire (pts (xy 146.05 106.045) (xy 146.05 109.855))
+    (stroke (width 0) (type default))
+  )
+  (wire (pts (xy 151.765 103.505) (xy 151.765 106.045))
+    (stroke (width 0) (type default))
+  )
   (wire (pts (xy 247.015 123.19) (xy 252.73 123.19))
     (stroke (width 0) (type default))
@@
   (wire (pts (xy 191.77 123.19) (xy 193.04 123.19))
     (stroke (width 0) (type default))
+  )
+  (text "Still not fucking working" (at 46.355 163.195 0)
+    (effects (font (size 10 10)) (justify left bottom))
   )
   (global_label "TXD" (shape output) (at 43.815 69.85 180) (fields_autoplaced)
@@
     )
   )
-  (global_label "VBUS" (shape input) (at 141.605 109.855 90) (fields_autoplaced)
+  (global_label "VBUS" (shape input) (at 156.845 106.045 0) (fields_autoplaced)
     (effects (font (size 1.27 1.27)) (justify left))
-    (property "Intersheetrefs" "${INTERSHEET_REFS}" (at 141.605 102.7048 90)
+    (property "Intersheetrefs" "${INTERSHEET_REFS}" (at 163.9952 106.045 0)
       (effects (font (size 1.27 1.27)) (justify left) hide)
     )
@@
     )
   )
+  (symbol (lib_id "Device:C") (at 146.05 99.695 0) (unit 1)
+    (in_bom yes) (on_board yes) (dnp no)
+    (property "Reference" "C3" (at 139.065 100.3331 0)
+      (effects (font (size 1.27 1.27)) (justify left))
+    )
+    (property "Value" "100nF" (at 139.065 102.87 0)
+      (effects (font (size 1.27 1.27)) (justify left))
+    )
+    (property "Footprint" "RevK:C_0402" (at 147.0152 103.505 0)
+      (effects (font (size 1.27 1.27)) hide)
+    )
+    (property "Datasheet" "~" (at 146.05 99.695 0)
+      (effects (font (size 1.27 1.27)) hide)
+    )
+    (pin "1")
+    (pin "2")
+    (instances
+      (project "Tas"
+        (path "/42713045-fffd-4b2d-ae1e-7232d705fb12"
+          (reference "C3") (unit 1)
+        )
+      )
+    )
+  )
   (symbol (lib_id "power:+3V3") (at 99.06 44.45 270) (unit 1)
     (in_bom yes) (on_board yes) (dnp no) (fields_autoplaced)
@@
     )
   )
-  (symbol (lib_id "Device:C") (at 139.065 99.695 0) (unit 1)
-    (in_bom yes) (on_board yes) (dnp no) (fields_autoplaced)
-    (property "Reference" "C2" (at 141.986 98.8603 0)
-      (effects (font (size 1.27 1.27)) (justify left))
-    )
-    (property "Value" "100nF" (at 141.986 101.3972 0)
-      (effects (font (size 1.27 1.27)) (justify left))
-    )
-    (property "Footprint" "RevK:C_0402" (at 140.0302 103.505 0)
-      (effects (font (size 1.27 1.27)) hide)
-    )
-    (property "Datasheet" "~" (at 139.065 99.695 0)
+  (symbol (lib_id "Device:C") (at 132.08 99.695 0) (unit 1)
+    (in_bom yes) (on_board yes) (dnp no)
+    (property "Reference" "C2" (at 125.73 100.3331 0)
+      (effects (font (size 1.27 1.27)) (justify left))
+    )
+    (property "Value" "10nF" (at 125.73 102.87 0)
+      (effects (font (size 1.27 1.27)) (justify left))
+    )
+    (property "Footprint" "RevK:C_0402" (at 133.0452 103.505 0)
+      (effects (font (size 1.27 1.27)) hide)
+    )
+    (property "Datasheet" "~" (at 132.08 99.695 0)
       (effects (font (size 1.27 1.27)) hide)
     )
@@
         (path "/825c70b0-4860-42b7-97dc-86bfa46e06fd"
           (reference "R7") (unit 1)
+        )
+      )
+    )
+  )
+  (symbol (lib_id "power:GND") (at 146.05 95.885 180) (unit 1)
+    (in_bom yes) (on_board yes) (dnp no) (fields_autoplaced)
+    (property "Reference" "#PWR023" (at 146.05 89.535 0)
+      (effects (font (size 1.27 1.27)) hide)
+    )
+    (property "Value" "GND" (at 146.05 91.94 0)
+      (effects (font (size 1.27 1.27)))
+    )
+    (property "Footprint" "" (at 146.05 95.885 0)
+      (effects (font (size 1.27 1.27)) hide)
+    )
+    (property "Datasheet" "" (at 146.05 95.885 0)
+      (effects (font (size 1.27 1.27)) hide)
+    )
+    (pin "1")
+    (instances
+      (project "Tas"
+        (path "/42713045-fffd-4b2d-ae1e-7232d705fb12"
+          (reference "#PWR023") (unit 1)
         )
       )
@@
         (path "/42713045-fffd-4b2d-ae1e-7232d705fb12"
           (reference "#PWR017") (unit 1)
+        )
+      )
+    )
+  )
+  (symbol (lib_id "Device:C") (at 151.765 99.695 0) (unit 1)
+    (in_bom yes) (on_board yes) (dnp no) (fields_autoplaced)
+    (property "Reference" "C4" (at 154.686 98.671 0)
+      (effects (font (size 1.27 1.27)) (justify left))
+    )
+    (property "Value" "22uF" (at 154.686 100.719 0)
+      (effects (font (size 1.27 1.27)) (justify left))
+    )
+    (property "Footprint" "RevK:C_0402" (at 152.7302 103.505 0)
+      (effects (font (size 1.27 1.27)) hide)
+    )
+    (property "Datasheet" "~" (at 151.765 99.695 0)
+      (effects (font (size 1.27 1.27)) hide)
+    )
+    (pin "1")
+    (pin "2")
+    (instances
+      (project "Tas"
+        (path "/42713045-fffd-4b2d-ae1e-7232d705fb12"
+          (reference "C4") (unit 1)
         )
       )
@@
     )
   )
-  (symbol (lib_id "power:GND") (at 139.065 95.885 180) (unit 1)
+  (symbol (lib_id "power:GND") (at 132.08 95.885 180) (unit 1)
     (in_bom yes) (on_board yes) (dnp no) (fields_autoplaced)
-    (property "Reference" "#PWR08" (at 139.065 89.535 0)
-      (effects (font (size 1.27 1.27)) hide)
-    )
-    (property "Value" "GND" (at 139.065 91.94 0)
-      (effects (font (size 1.27 1.27)))
-    )
-    (property "Footprint" "" (at 139.065 95.885 0)
-      (effects (font (size 1.27 1.27)) hide)
-    )
-    (property "Datasheet" "" (at 139.065 95.885 0)
+    (property "Reference" "#PWR08" (at 132.08 89.535 0)
+      (effects (font (size 1.27 1.27)) hide)
+    )
+    (property "Value" "GND" (at 132.08 91.94 0)
+      (effects (font (size 1.27 1.27)))
+    )
+    (property "Footprint" "" (at 132.08 95.885 0)
+      (effects (font (size 1.27 1.27)) hide)
+    )
+    (property "Datasheet" "" (at 132.08 95.885 0)
       (effects (font (size 1.27 1.27)) hide)
     )
@@
         )
       )
+    )
+  )
+  (symbol (lib_id "power:GND") (at 151.765 95.885 180) (unit 1)
+    (in_bom yes) (on_board yes) (dnp no) (fields_autoplaced)
+    (property "Reference" "#PWR024" (at 151.765 89.535 0)
+      (effects (font (size 1.27 1.27)) hide)
+    )
+    (property "Value" "GND" (at 151.765 91.94 0)
+      (effects (font (size 1.27 1.27)))
+    )
+    (property "Footprint" "" (at 151.765 95.885 0)
+      (effects (font (size 1.27 1.27)) hide)
+    )
+    (property "Datasheet" "" (at 151.765 95.885 0)
+      (effects (font (size 1.27 1.27)) hide)
+    )
+    (pin "1")
+    (instances
+      (project "Tas"
+        (path "/42713045-fffd-4b2d-ae1e-7232d705fb12"
+          (reference "#PWR024") (unit 1)
+        )
+      )
