File: PCB/ShellyMini/ShellyMini.kicad_pcb (KiCad board)
At the start: 2 copper layers, 206 x 50 mm, 40 parts, among them J1 Shelly

Commit message: Correct bottom plate
Other:
- outline, holes or cut-outs redrawn

Commit message: Tidy up a lot
Parts:
- added H25: MountingHole, MountingHole:MountingHole_3.2mm_M3, F.Cu at (52.0, 80.0)
- added H26: MountingHole, MountingHole:MountingHole_3.2mm_M3, F.Cu at (92.0, 80.0)
- added H27: MountingHole, MountingHole:MountingHole_3.2mm_M3, F.Cu at (92.0, 120.0)
- added H28: MountingHole, MountingHole:MountingHole_3.2mm_M3, F.Cu at (52.0, 120.0)
Other:
- outline, holes or cut-outs redrawn
- board text added: "1"
- board text added: "2"
- board text added: "3"
- board text added: "4"
- board text added: "www.me.uk"

Commit message: More spacers
Parts:
- added Z4: Hidden, RevK:PCB-Join, F.Cu at (98.0, 110.0)
- added Z5: Hidden, RevK:PCB-Join, F.Cu at (150.0, 90.0)
- added Z6: Hidden, RevK:PCB-Join, F.Cu at (202.0, 90.0)
- moved Z3 10.9 mm to (98.0, 89.1)
- moved Z1 10.0 mm to (150.0, 110.0)
- moved Z2 10.0 mm to (202.0, 110.0)
Other:
- outline, holes or cut-outs redrawn

Commit message: Tweaks
Parts:
- moved H23 1.00 mm to (72.0, 80.0)
- moved H9 1.00 mm to (228.0, 80.0)
Other:
- outline, holes or cut-outs redrawn
- board text added: "3V3"
- board text added: "Boot"
- board text added: "EN"
- board text added: "Rx"
- board text added: "Tx"
- board text added: "⏚"

Commit message: Revised
Parts:
- removed H17, H18, H19, H20, H21, H22, H23, H24: MountingHole, MountingHole:MountingHole_3.2mm_M3
- added Z7: Hidden, RevK:PCB-Join, F.Cu at (134.0, 126.0)
- added Z8: Hidden, RevK:PCB-Join, F.Cu at (114.0, 126.0)
- moved H10 116.3 mm to (52.0, 152.0)
- moved H11 116.3 mm to (124.0, 172.0)
- moved H12 116.3 mm to (144.0, 152.0)
- moved H13 116.3 mm to (52.0, 132.0)
- moved H14 116.3 mm to (92.0, 132.0)
- moved H15 116.3 mm to (52.0, 172.0)
- moved H16 116.3 mm to (92.0, 172.0)
- moved H5 116.3 mm to (72.0, 132.0)
- moved H6 116.3 mm to (104.0, 152.0)
- moved H7 116.3 mm to (92.0, 152.0)
- moved H8 116.3 mm to (72.0, 172.0)
- moved H9 116.3 mm to (124.0, 132.0)
- moved TP1 116.3 mm to (109.5, 148.8)
- moved TP10 116.3 mm to (57.5, 154.9)
- moved TP11 116.3 mm to (57.5, 156.3)
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Other:
- board size 206 x 50 mm -> 102 x 102 mm
- board text added: "3A"
- board text added: "3B"
- board text removed: "3"
- board text removed: "4"
