File: PCB/ShellyMini/ShellyMini.kicad_sch (KiCad schematic)
At the start: 40 parts, among them J1 Shelly

Commit message: Tidy up a lot
Parts:
- added H25, H26, H27, H28: MountingHole, MountingHole:MountingHole_3.2mm_M3, symbol Mechanical:MountingHole
Changed lines of the file:
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@@
+    )
+  )
+  (symbol (lib_id "Mechanical:MountingHole") (at 74.295 63.5 0) (unit 1)
+    (in_bom yes) (on_board yes) (dnp no) (fields_autoplaced)
+    (property "Reference" "H28" (at 76.835 62.2879 0)
+      (effects (font (size 1.27 1.27)) (justify left))
+    )
+    (property "Value" "MountingHole" (at 76.835 64.7121 0)
+      (effects (font (size 1.27 1.27)) (justify left))
+    )
+    (property "Footprint" "MountingHole:MountingHole_3.2mm_M3" (at 74.295 63.5 0)
+      (effects (font (size 1.27 1.27)) hide)
+    )
+    (property "Datasheet" "~" (at 74.295 63.5 0)
+      (effects (font (size 1.27 1.27)) hide)
+    )
+    (instances
+      (project "ShellyMini"
+        (path "/eb815f10-ee47-480a-bf97-ce549d1e9a75"
+          (reference "H28") (unit 1)
+        )
+      )
     )
   )
@@
     )
   )
+  (symbol (lib_id "Mechanical:MountingHole") (at 73.025 95.885 0) (unit 1)
+    (in_bom yes) (on_board yes) (dnp no) (fields_autoplaced)
+    (property "Reference" "H27" (at 75.565 94.6729 0)
+      (effects (font (size 1.27 1.27)) (justify left))
+    )
+    (property "Value" "MountingHole" (at 75.565 97.0971 0)
+      (effects (font (size 1.27 1.27)) (justify left))
+    )
+    (property "Footprint" "MountingHole:MountingHole_3.2mm_M3" (at 73.025 95.885 0)
+      (effects (font (size 1.27 1.27)) hide)
+    )
+    (property "Datasheet" "~" (at 73.025 95.885 0)
+      (effects (font (size 1.27 1.27)) hide)
+    )
+    (instances
+      (project "ShellyMini"
+        (path "/eb815f10-ee47-480a-bf97-ce549d1e9a75"
+          (reference "H27") (unit 1)
+        )
+      )
+    )
+  )
   (symbol (lib_id "Mechanical:MountingHole") (at 73.025 90.805 0) (unit 1)
     (in_bom yes) (on_board yes) (dnp no) (fields_autoplaced)
@@
         )
       )
+    )
+  )
+  (symbol (lib_id "Mechanical:MountingHole") (at 27.94 63.5 0) (unit 1)
+    (in_bom yes) (on_board yes) (dnp no) (fields_autoplaced)
+    (property "Reference" "H26" (at 30.48 62.2879 0)
+      (effects (font (size 1.27 1.27)) (justify left))
+    )
+    (property "Value" "MountingHole" (at 30.48 64.7121 0)
+      (effects (font (size 1.27 1.27)) (justify left))
+    )
+    (property "Footprint" "MountingHole:MountingHole_3.2mm_M3" (at 27.94 63.5 0)
+      (effects (font (size 1.27 1.27)) hide)
+    )
+    (property "Datasheet" "~" (at 27.94 63.5 0)
+      (effects (font (size 1.27 1.27)) hide)
+    )
+    (instances
+      (project "ShellyMini"
+        (path "/eb815f10-ee47-480a-bf97-ce549d1e9a75"
+          (reference "H26") (unit 1)
+        )
+      )
+    )
+  )
+  (symbol (lib_id "Mechanical:MountingHole") (at 27.305 94.615 0) (unit 1)
+    (in_bom yes) (on_board yes) (dnp no) (fields_autoplaced)
+    (property "Reference" "H25" (at 29.845 93.4029 0)
+      (effects (font (size 1.27 1.27)) (justify left))
+    )
+    (property "Value" "MountingHole" (at 29.845 95.8271 0)
+      (effects (font (size 1.27 1.27)) (justify left))
+    )
+    (property "Footprint" "MountingHole:MountingHole_3.2mm_M3" (at 27.305 94.615 0)
+      (effects (font (size 1.27 1.27)) hide)
+    )
+    (property "Datasheet" "~" (at 27.305 94.615 0)
+      (effects (font (size 1.27 1.27)) hide)
+    )
+    (instances
+      (project "ShellyMini"
+        (path "/eb815f10-ee47-480a-bf97-ce549d1e9a75"
+          (reference "H25") (unit 1)
+        )
+      )

Commit message: More spacers
Parts:
- added Z4, Z5, Z6: Hidden, RevK:PCB-Join, symbol RevK:Hidden
Other:
- moved on the sheet: Z1, Z2, Z3
Changed lines of the file:
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@@
     )
   )
-  (symbol (lib_id "RevK:Hidden") (at 180.975 71.755 0) (unit 1)
+  (symbol (lib_id "RevK:Hidden") (at 204.47 116.84 0) (unit 1)
     (in_bom no) (on_board yes) (dnp no) (fields_autoplaced)
-    (property "Reference" "Z1" (at 182.3212 70.5429 0)
-      (effects (font (size 1.27 1.27)) (justify left))
-    )
-    (property "Value" "Hidden" (at 182.3212 72.9671 0)
-      (effects (font (size 1.27 1.27)) (justify left))
-    )
-    (property "Footprint" "RevK:PCB-Join" (at 180.975 69.85 0)
-      (effects (font (size 1.27 1.27)) hide)
-    )
-    (property "Datasheet" "" (at 180.975 71.755 0)
-      (effects (font (size 1.27 1.27)) hide)
-    )
-    (property "Part No" "" (at 180.975 71.755 0)
-      (effects (font (size 1.27 1.27)) hide)
-    )
-    (property "Note" "" (at 180.975 71.755 0)
+    (property "Reference" "Z1" (at 205.8162 115.6279 0)
+      (effects (font (size 1.27 1.27)) (justify left))
+    )
+    (property "Value" "Hidden" (at 205.8162 118.0521 0)
+      (effects (font (size 1.27 1.27)) (justify left))
+    )
+    (property "Footprint" "RevK:PCB-Join" (at 204.47 114.935 0)
+      (effects (font (size 1.27 1.27)) hide)
+    )
+    (property "Datasheet" "" (at 204.47 116.84 0)
+      (effects (font (size 1.27 1.27)) hide)
+    )
+    (property "Part No" "" (at 204.47 116.84 0)
+      (effects (font (size 1.27 1.27)) hide)
+    )
+    (property "Note" "" (at 204.47 116.84 0)
       (effects (font (size 1.27 1.27)) hide)
     )
@@
     )
   )
+  (symbol (lib_id "RevK:Hidden") (at 215.265 127.635 0) (unit 1)
+    (in_bom no) (on_board yes) (dnp no) (fields_autoplaced)
+    (property "Reference" "Z6" (at 216.6112 126.4229 0)
+      (effects (font (size 1.27 1.27)) (justify left))
+    )
+    (property "Value" "Hidden" (at 216.6112 128.8471 0)
+      (effects (font (size 1.27 1.27)) (justify left))
+    )
+    (property "Footprint" "RevK:PCB-Join" (at 215.265 125.73 0)
+      (effects (font (size 1.27 1.27)) hide)
+    )
+    (property "Datasheet" "" (at 215.265 127.635 0)
+      (effects (font (size 1.27 1.27)) hide)
+    )
+    (property "Part No" "" (at 215.265 127.635 0)
+      (effects (font (size 1.27 1.27)) hide)
+    )
+    (property "Note" "" (at 215.265 127.635 0)
+      (effects (font (size 1.27 1.27)) hide)
+    )
+    (pin "~")
+    (instances
+      (project "ShellyMini"
+        (path "/eb815f10-ee47-480a-bf97-ce549d1e9a75"
+          (reference "Z6") (unit 1)
+        )
+      )
+    )
+  )
   (symbol (lib_id "Mechanical:MountingHole") (at 90.17 65.405 0) (unit 1)
     (in_bom yes) (on_board yes) (dnp no) (fields_autoplaced)
@@
     )
   )
-  (symbol (lib_id "RevK:Hidden") (at 267.335 132.715 0) (unit 1)
+  (symbol (lib_id "RevK:Hidden") (at 204.47 127.635 0) (unit 1)
     (in_bom no) (on_board yes) (dnp no) (fields_autoplaced)
-    (property "Reference" "Z3" (at 268.6812 131.5029 0)
-      (effects (font (size 1.27 1.27)) (justify left))
-    )
-    (property "Value" "Hidden" (at 268.6812 133.9271 0)
-      (effects (font (size 1.27 1.27)) (justify left))
-    )
-    (property "Footprint" "RevK:PCB-Join" (at 267.335 130.81 0)
-      (effects (font (size 1.27 1.27)) hide)
-    )
-    (property "Datasheet" "" (at 267.335 132.715 0)
-      (effects (font (size 1.27 1.27)) hide)
-    )
-    (property "Part No" "" (at 267.335 132.715 0)
-      (effects (font (size 1.27 1.27)) hide)
-    )
-    (property "Note" "" (at 267.335 132.715 0)
+    (property "Reference" "Z3" (at 205.8162 126.4229 0)
+      (effects (font (size 1.27 1.27)) (justify left))
+    )
+    (property "Value" "Hidden" (at 205.8162 128.8471 0)
+      (effects (font (size 1.27 1.27)) (justify left))
+    )
+    (property "Footprint" "RevK:PCB-Join" (at 204.47 125.73 0)
+      (effects (font (size 1.27 1.27)) hide)
+    )
+    (property "Datasheet" "" (at 204.47 127.635 0)
+      (effects (font (size 1.27 1.27)) hide)
+    )
+    (property "Part No" "" (at 204.47 127.635 0)
+      (effects (font (size 1.27 1.27)) hide)
+    )
+    (property "Note" "" (at 204.47 127.635 0)
       (effects (font (size 1.27 1.27)) hide)
     )
@@
     )
   )
+  (symbol (lib_id "RevK:Hidden") (at 215.265 116.84 0) (unit 1)
+    (in_bom no) (on_board yes) (dnp no) (fields_autoplaced)
+    (property "Reference" "Z4" (at 216.6112 115.6279 0)
+      (effects (font (size 1.27 1.27)) (justify left))
+    )
+    (property "Value" "Hidden" (at 216.6112 118.0521 0)
+      (effects (font (size 1.27 1.27)) (justify left))
+    )
+    (property "Footprint" "RevK:PCB-Join" (at 215.265 114.935 0)
+      (effects (font (size 1.27 1.27)) hide)
+    )
+    (property "Datasheet" "" (at 215.265 116.84 0)
+      (effects (font (size 1.27 1.27)) hide)
+    )
+    (property "Part No" "" (at 215.265 116.84 0)
+      (effects (font (size 1.27 1.27)) hide)
+    )
+    (property "Note" "" (at 215.265 116.84 0)
+      (effects (font (size 1.27 1.27)) hide)
+    )
+    (pin "~")
+    (instances
+      (project "ShellyMini"
+        (path "/eb815f10-ee47-480a-bf97-ce549d1e9a75"
+          (reference "Z4") (unit 1)
+        )
+      )
+    )
+  )
   (symbol (lib_id "Mechanical:MountingHole") (at 89.535 96.52 0) (unit 1)
     (in_bom yes) (on_board yes) (dnp no) (fields_autoplaced)
@@
     )
   )
-  (symbol (lib_id "RevK:Hidden") (at 253.365 133.985 0) (unit 1)
+  (symbol (lib_id "RevK:Hidden") (at 204.47 122.555 0) (unit 1)
     (in_bom no) (on_board yes) (dnp no) (fields_autoplaced)
-    (property "Reference" "Z2" (at 254.7112 132.7729 0)
-      (effects (font (size 1.27 1.27)) (justify left))
-    )
-    (property "Value" "Hidden" (at 254.7112 135.1971 0)
-      (effects (font (size 1.27 1.27)) (justify left))
-    )
-    (property "Footprint" "RevK:PCB-Join" (at 253.365 132.08 0)
-      (effects (font (size 1.27 1.27)) hide)
-    )
-    (property "Datasheet" "" (at 253.365 133.985 0)
-      (effects (font (size 1.27 1.27)) hide)
-    )
-    (property "Part No" "" (at 253.365 133.985 0)
-      (effects (font (size 1.27 1.27)) hide)
-    )
-    (property "Note" "" (at 253.365 133.985 0)
+    (property "Reference" "Z2" (at 205.8162 121.3429 0)
+      (effects (font (size 1.27 1.27)) (justify left))
+    )
+    (property "Value" "Hidden" (at 205.8162 123.7671 0)
+      (effects (font (size 1.27 1.27)) (justify left))
+    )
+    (property "Footprint" "RevK:PCB-Join" (at 204.47 120.65 0)
+      (effects (font (size 1.27 1.27)) hide)
+    )
+    (property "Datasheet" "" (at 204.47 122.555 0)
+      (effects (font (size 1.27 1.27)) hide)
+    )
+    (property "Part No" "" (at 204.47 122.555 0)
+      (effects (font (size 1.27 1.27)) hide)
+    )
+    (property "Note" "" (at 204.47 122.555 0)
       (effects (font (size 1.27 1.27)) hide)
     )
@@
         )
       )
+    )
+  )
+  (symbol (lib_id "RevK:Hidden") (at 215.265 122.555 0) (unit 1)
+    (in_bom no) (on_board yes) (dnp no) (fields_autoplaced)
+    (property "Reference" "Z5" (at 216.6112 121.3429 0)
+      (effects (font (size 1.27 1.27)) (justify left))
+    )
+    (property "Value" "Hidden" (at 216.6112 123.7671 0)
+      (effects (font (size 1.27 1.27)) (justify left))
+    )
+    (property "Footprint" "RevK:PCB-Join" (at 215.265 120.65 0)
+      (effects (font (size 1.27 1.27)) hide)
+    )
+    (property "Datasheet" "" (at 215.265 122.555 0)
+      (effects (font (size 1.27 1.27)) hide)
+    )
+    (property "Part No" "" (at 215.265 122.555 0)
+      (effects (font (size 1.27 1.27)) hide)
+    )
+    (property "Note" "" (at 215.265 122.555 0)
+      (effects (font (size 1.27 1.27)) hide)
+    )
+    (pin "~")
+    (instances
+      (project "ShellyMini"
+        (path "/eb815f10-ee47-480a-bf97-ce549d1e9a75"
+          (reference "Z5") (unit 1)
+        )
+      )

Commit message: Revised
Parts:
- removed H17, H18, H19, H20, H21, H22, H23, H24: MountingHole, MountingHole:MountingHole_3.2mm_M3, symbol Mechanical:MountingHole
- added Z7, Z8: Hidden, RevK:PCB-Join, symbol RevK:Hidden
Other:
- moved on the sheet: Z4, Z5, Z6
