File: PCB/TasPanel/Tas.kicad_sch (KiCad schematic)
At the start: 34 parts, among them J1 Shelly 1, J2 Conn_01x07, J3 USB-C-Socket-V, Q1 PMF170XP,115, Q2 PMF250XNEX, U1 FT231XQ, U3 MD8942

Commit message: Panel and non panel
Parts:
- added PCB1: 70x70, RevK:PCB7070, symbol RevK:PCB
- added V2, V3: ~, RevK:VCUT70N, symbol RevK:VCUT
Changed lines of the file:
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@@
+	)
+	(symbol
+		(lib_id "RevK:VCUT")
+		(at 249.555 175.895 180)
+		(unit 1)
+		(exclude_from_sim yes)
+		(in_bom no)
+		(on_board yes)
+		(dnp no)
+		(fields_autoplaced yes)
+		(property "Reference" "V3"
+			(at 249.555 177.165 0)
+			(effects
+				(font
+					(size 1.27 1.27)
+				)
+				(hide yes)
+			)
+		)
+		(property "Value" "~"
+			(at 249.555 175.895 0)
+			(effects
+				(font
+					(size 1.27 1.27)
+				)
+			)
+		)
+		(property "Footprint" "RevK:VCUT70N"
+			(at 249.555 174.625 0)
+			(effects
+				(font
+					(size 1.27 1.27)
+				)
+				(hide yes)
+			)
+		)
+		(property "Datasheet" ""
+			(at 249.555 175.895 0)
+			(effects
+				(font
+					(size 1.27 1.27)
+				)
+				(hide yes)
+			)
+		)
+		(property "Description" ""
+			(at 249.555 175.895 0)
+			(effects
+				(font
+					(size 1.27 1.27)
+				)
+				(hide yes)
+			)
+		)
+		(instances
+			(project "Tas"
+				(path "/42713045-fffd-4b2d-ae1e-7232d705fb12"
+					(reference "V3")
+					(unit 1)
+				)
+			)
+		)
 	)
 	(symbol
@@
 	)
 	(symbol
+		(lib_id "RevK:VCUT")
+		(at 249.555 169.545 180)
+		(unit 1)
+		(exclude_from_sim yes)
+		(in_bom no)
+		(on_board yes)
+		(dnp no)
+		(fields_autoplaced yes)
+		(property "Reference" "V2"
+			(at 249.555 170.815 0)
+			(effects
+				(font
+					(size 1.27 1.27)
+				)
+				(hide yes)
+			)
+		)
+		(property "Value" "~"
+			(at 249.555 169.545 0)
+			(effects
+				(font
+					(size 1.27 1.27)
+				)
+			)
+		)
+		(property "Footprint" "RevK:VCUT70N"
+			(at 249.555 168.275 0)
+			(effects
+				(font
+					(size 1.27 1.27)
+				)
+				(hide yes)
+			)
+		)
+		(property "Datasheet" ""
+			(at 249.555 169.545 0)
+			(effects
+				(font
+					(size 1.27 1.27)
+				)
+				(hide yes)
+			)
+		)
+		(property "Description" ""
+			(at 249.555 169.545 0)
+			(effects
+				(font
+					(size 1.27 1.27)
+				)
+				(hide yes)
+			)
+		)
+		(instances
+			(project "Tas"
+				(path "/42713045-fffd-4b2d-ae1e-7232d705fb12"
+					(reference "V2")
+					(unit 1)
+				)
+			)
+		)
+	)
+	(symbol
 		(lib_id "power:+3.3V")
 		(at 57.785 52.07 0)
@@
 					(unit 1)
 				)
+			)
+		)
+	)
+	(symbol
+		(lib_id "RevK:PCB")
+		(at 249.555 172.72 0)
+		(unit 1)
+		(exclude_from_sim no)
+		(in_bom no)
+		(on_board yes)
+		(dnp no)
+		(property "Reference" "PCB1"
+			(at 249.555 182.88 0)
+			(effects
+				(font
+					(size 1.27 1.27)
+				)
+				(hide yes)
+			)
+		)
+		(property "Value" "70x70"
+			(at 249.555 172.72 0)
+			(effects
+				(font
+					(size 1.27 1.27)
+				)
+			)
+		)
+		(property "Footprint" "RevK:PCB7070"
+			(at 249.555 167.005 0)
+			(effects
+				(font
+					(size 1.27 1.27)
+				)
+				(hide yes)
+			)
+		)
+		(property "Datasheet" ""
+			(at 249.555 172.72 0)
+			(effects
+				(font
+					(size 1.27 1.27)
+				)
+				(hide yes)
+			)
+		)
+		(property "Description" ""
+			(at 249.555 172.72 0)
+			(effects
+				(font
+					(size 1.27 1.27)
+				)
+				(hide yes)
+			)
+		)
+		(instances
+			(project "Tas"
+				(path "/42713045-fffd-4b2d-ae1e-7232d705fb12"
+					(reference "PCB1")
+					(unit 1)
+				)

Commit message: PCB Update
Parts:
- C6: LCSC Part # C194427 -> (none); MPN (none) -> C194427
- C7: LCSC Part # C1691 -> (none); MPN (none) -> C1691
- D1, D2, D3, D5: LCSC Part # C5137770 -> (none); MPN (none) -> C5137770
- D4: LCSC Part # C264508 -> (none); MPN (none) -> C264508
- J1: LCSC Part # C225491 -> (none); MPN (none) -> C225491
- J2: JLCPCB Rotation Offset 90 -> (none); LCSC Part # C2832274 -> (none); MPN (none) -> C2832274
- J3: LCSC Part # C709357 -> (none); MPN (none) -> C709357
- U1: JLCPCB Rotation Offset -90 -> (none); LCSC Part # C132159 -> (none); MPN (none) -> C132159
- U3: LCSC Part # C2684786 -> (none); MPN (none) -> C2684786
- renumbered C27 to C10, C1 to C2, C2 to C3, C2 to C4, C1 to C9
Changed lines of the file:
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@@
 (kicad_sch
-	(version 20231120)
+	(version 20241209)
 	(generator "eeschema")
-	(generator_version "8.0")
+	(generator_version "9.0")
 	(paper "A4")
 	(title_block
@@
 		(comment 2 "www.me.uk")
 	)
+	(text "Configure FTDI\n- Inverted RTS\n- CBUS modes for LEDs, suggest :-\n- CBUS0 mode 1\n- CBUS1 mode 2\n- CBUS3 mode 9"
+		(exclude_from_sim no)
+		(at 177.165 116.205 0)
+		(effects
+			(font
+				(size 2.54 2.54)
+			)
+			(justify left bottom)
+		)
+	)
 	(junction
 		(at 114.935 117.475)
@@
 		)
 	)
-	(text "Configure FTDI\n- Inverted RTS\n- CBUS modes for LEDs, suggest :-\n- CBUS0 mode 1\n- CBUS1 mode 2\n- CBUS3 mode 9"
-		(exclude_from_sim no)
-		(at 177.165 116.205 0)
-		(effects
-			(font
-				(size 2.54 2.54)
-			)
-			(justify left bottom)
-		)
-	)
 	(global_label "TXD"
 		(shape output)
@@
 			)
 		)
-		(property "Description" ""
+		(property "Description" "Generic connector, single row, 01x05, script generated (kicad-library-utils/schlib/autogen/connector/)"
 			(at 73.66 43.18 0)
 			(effects
@@
 			)
 		)
-		(property "LCSC Part #" "C225491"
+		(property "MPN" "C225491"
 			(at 73.66 43.18 0)
 			(effects
@@
 			)
 		)
-		(property "Description" ""
+		(property "Description" "Full Speed USB to Full Handshake UART, QFN-20"
 			(at 142.875 132.715 0)
 			(effects
@@
 			)
 		)
-		(property "LCSC Part #" "C132159"
-			(at 142.875 132.715 0)
-			(effects
-				(font
-					(size 1.27 1.27)
-				)
-				(hide yes)
-			)
-		)
-		(property "JLCPCB Rotation Offset" "-90"
+		(property "MPN" "C132159"
 			(at 142.875 132.715 0)
 			(effects
@@
 		(dnp no)
 		(fields_autoplaced yes)
-		(property "Reference" "C2"
+		(property "Reference" "C3"
 			(at 60.706 54.856 0)
 			(effects
@@
 			)
 		)
-		(property "LCSC Part #" "C264508"
+		(property "MPN" "C264508"
 			(at 190.5 144.145 0)
 			(effects
@@
 		(on_board yes)
 		(dnp no)
-		(property "Reference" "C2"
+		(property "Reference" "C4"
 			(at 233.045 74.152 0)
 			(effects
@@
 		(dnp no)
 		(fields_autoplaced yes)
-		(property "Reference" "#PWR011"
+		(property "Reference" "#PWR024"
 			(at 51.435 66.04 0)
 			(effects
@@
 			)
 		)
-		(property "LCSC Part #" "C2832274"
-			(at 73.66 72.39 0)
-			(effects
-				(font
-					(size 1.27 1.27)
-				)
-				(hide yes)
-			)
-		)
-		(property "JLCPCB Rotation Offset" "90"
+		(property "MPN" "C2832274"
 			(at 73.66 72.39 0)
 			(effects
@@
 		(on_board yes)
 		(dnp no)
-		(property "Reference" "C27"
+		(property "Reference" "C10"
 			(at 255.905 74.295 0)
 			(effects
@@
 		(dnp no)
 		(fields_autoplaced yes)
-		(property "Reference" "#PWR012"
+		(property "Reference" "#PWR023"
 			(at 57.785 55.88 0)
 			(effects
@@
 			)
 		)
-		(property "LCSC Part #" "C5137770"
+		(property "MPN" "C5137770"
 			(at 65.405 125.73 0)
 			(effects
@@
 			)
 		)
-		(property "LCSC Part #" "C194427"
+		(property "MPN" "C194427"
 			(at 229.235 41.275 0)
 			(effects
@@
 		(on_board yes)
 		(dnp no)
-		(property "Reference" "#PWR038"
+		(property "Reference" "#PWR032"
 			(at 248.92 85.09 0)
 			(effects
@@
 		(on_board yes)
 		(dnp no)
-		(property "Reference" "C1"
+		(property "Reference" "C9"
 			(at 220.98 73.517 0)
 			(effects
@@
 			)
 		)
-		(property "Description" ""
+		(property "Description" "Regulator and associated components."
 			(at 208.28 47.625 0)
 			(effects
@@
 			)
 		)
-		(property "LCSC Part #" "C2684786"
-			(at 208.28 74.295 0)
+		(property "MPN" "C2684786"
+			(at 208.28 47.625 0)
 			(effects
 				(font
@@
 		(dnp no)
 		(fields_autoplaced yes)
-		(property "Reference" "#PWR08"
+		(property "Reference" "#PWR021"
 			(at 51.435 55.88 0)
 			(effects
@@
 			)
 		)
-		(property "LCSC Part #" "C5137770"
+		(property "MPN" "C5137770"
 			(at 65.405 120.65 0)
 			(effects
@@
 			)
 		)
-		(property "LCSC Part #" "C5137770"
+		(property "MPN" "C5137770"
 			(at 65.405 109.22 0)
 			(effects
@@
 			)
 		)
-		(property "LCSC Part #" "C5137770"
+		(property "MPN" "C5137770"
 			(at 65.405 114.935 0)
 			(effects
@@
 		(dnp no)
 		(fields_autoplaced yes)
-		(property "Reference" "#PWR013"
+		(property "Reference" "#PWR029"
 			(at 57.785 66.04 0)
 			(effects
@@
 			)
 		)
-		(property "LCSC Part #" "C1691"
+		(property "MPN" "C1691"
 			(at 229.235 43.18 0)
 			(effects
@@
 		(on_board yes)
 		(dnp no)
-		(property "Reference" "C1"
+		(property "Reference" "C2"
 			(at 42.545 54.467 0)
 			(effects
@@
 			)
 		)
-		(property "Description" ""
+		(property "Description" "USB 2.0-only Type-C Receptacle connector"
 			(at 138.43 60.96 0)
 			(effects
@@
 			)
 		)
-		(property "LCSC Part #" "C709357"
+		(property "MPN" "C709357"
 			(at 138.43 60.96 0)
 			(effects
@@
 		)
 	)
+	(embedded_fonts no)
 )
